File: hardware/MacSAO.kicad_pcb (KiCad board)
At the start: 2 copper layers, 24.9 x 33.6 mm, 10 parts, among them J1 2x3 SMD Pin Header, J2 Display Connector, SW1 EVQP7J01P, U1 A-SP110GHC-C01-2C, U2 CH32V003J4M6_C5346354, U3 ZD24C08A-STGMT

Commit message: Updates version 1.3, adds back in detail line
Other:
- board text added: "v1.3"
- board text removed: "v1.2"
