File: hardware/MacSAO.kicad_sch (KiCad schematic)
At the start: 10 parts, among them J1 2x3 SMD Pin Header, J2 Display Connector, SW1 EVQP7J01P, U1 A-SP110GHC-C01-2C, U2 CH32V003J4M6_C5346354, U3 ZD24C08A-STGMT

Commit message: Updates version 1.3, adds back in detail line
Other:
- company: (none) -> Conductive Resistance
- title: (none) -> Mac SAO
Changed lines of the file:
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@@
 (kicad_sch
-	(version 20231120)
+	(version 20250114)
 	(generator "eeschema")
-	(generator_version "8.0")
+	(generator_version "9.0")
 	(paper "A4")
+	(title_block
+		(title "Mac SAO")
+		(date "2026-04-18")
+		(rev "1.3")
+		(company "Conductive Resistance")
+	)
 	(junction
 		(at 105.41 31.75)
@@
 	(label "VCC"
 		(at 74.295 62.865 0)
-		(fields_autoplaced yes)
 		(effects
 			(font
@@
 	(label "ProgramEN"
 		(at 33.655 32.385 0)
-		(fields_autoplaced yes)
 		(effects
 			(font
@@
 	(label "ProgramEN"
 		(at 79.375 88.265 180)
-		(fields_autoplaced yes)
 		(effects
 			(font
@@
 	(label "SDA"
 		(at 33.655 27.305 0)
-		(fields_autoplaced yes)
 		(effects
 			(font
@@
 	(label "SoftSDA"
 		(at 73.66 24.13 0)
-		(fields_autoplaced yes)
 		(effects
 			(font
@@
 	(label "SDA"
 		(at 74.295 60.325 0)
-		(fields_autoplaced yes)
 		(effects
 			(font
@@
 	(label "GND"
 		(at 99.695 31.75 180)
-		(fields_autoplaced yes)
 		(effects
 			(font
@@
 	(label "SWIO"
 		(at 84.455 88.265 0)
-		(fields_autoplaced yes)
 		(effects
 			(font
@@
 	(label "VCC"
 		(at 100.0711 26.6524 180)
-		(fields_autoplaced yes)
 		(effects
 			(font
@@
 	(label "SoftSCL"
 		(at 74.295 65.405 0)
-		(fields_autoplaced yes)
 		(effects
 			(font
@@
 	(label "SoftSCL"
 		(at 73.66 26.67 0)
-		(fields_autoplaced yes)
 		(effects
 			(font
@@
 	(label "SWIO"
 		(at 74.295 52.705 0)
-		(fields_autoplaced yes)
 		(effects
 			(font
@@
 	(label "GPIO2"
 		(at 107.315 48.895 180)
-		(fields_autoplaced yes)
 		(effects
 			(font
@@
 	(label "SoftSDA"
 		(at 74.295 70.485 0)
-		(fields_autoplaced yes)
 		(effects
 			(font
@@
 	(label "GPIO2"
 		(at 33.655 34.925 0)
-		(fields_autoplaced yes)
 		(effects
 			(font
@@
 	(label "GND"
 		(at 74.295 67.945 0)
-		(fields_autoplaced yes)
 		(effects
 			(font
@@
 	(label "SCL"
 		(at 33.655 29.845 0)
-		(fields_autoplaced yes)
 		(effects
 			(font
@@
 	(label "SoftSDA"
 		(at 31.115 90.805 180)
-		(fields_autoplaced yes)
 		(effects
 			(font
@@
 	(label "GPIO2"
 		(at 74.295 55.245 0)
-		(fields_autoplaced yes)
 		(effects
 			(font
@@
 	(label "SCL"
 		(at 74.295 57.785 0)
-		(fields_autoplaced yes)
 		(effects
 			(font
@@
 	(label "SoftSCL"
 		(at 31.115 85.725 180)
-		(fields_autoplaced yes)
 		(effects
 			(font
@@
 		)
 		(instances
-			(project ""
+			(project "MacSAO"
 				(path "/e8b57aea-3d1d-4a23-81df-12a34aed9b0c"
 					(reference "JP1")
@@
 		)
 		(instances
-			(project ""
+			(project "MacSAO"
 				(path "/e8b57aea-3d1d-4a23-81df-12a34aed9b0c"
 					(reference "U3")
@@
 		)
 		(instances
-			(project ""
+			(project "MacSAO"
 				(path "/e8b57aea-3d1d-4a23-81df-12a34aed9b0c"
 					(reference "R1")
@@
 		)
 		(instances
-			(project ""
+			(project "MacSAO"
 				(path "/e8b57aea-3d1d-4a23-81df-12a34aed9b0c"
 					(reference "SW1")
@@
 		)
 		(instances
-			(project ""
+			(project "MacSAO"
 				(path "/e8b57aea-3d1d-4a23-81df-12a34aed9b0c"
 					(reference "U1")
@@
 		)
 	)
+	(embedded_fonts no)
 )
